Commit message: Commit

File: src/slambot_description/urdf/pentaslam.urdf.xacro (robot description, xacro)
@@ -1,6 +1,8 @@
 <?xml version="1.0"?>
-<robot name="pentaslam"
+<robot name="slambot"
     xmlns:xacro="http://www.ros.org/wiki/xacro">
-    <xacro:include filename="$(find pentaslam_description)/urdf/pentaslam_gazebo.xacro"/>
+    <xacro:arg name="is_sim" default="true"/>
+    <xacro:include filename="$(find slambot_description)/urdf/pentaslam_gazebo.xacro"/>
+    <xacro:include filename="$(find slambot_description)/urdf/pentaslam_ros2_control.xacro"/>
     <xacro:property name="PI" value="3.14159"/>
     <xacro:property name="effort" value="30"/>
@@ -23,5 +25,5 @@
             <origin xyz="0 0 0" rpy="0 0 0"/>
             <geometry>
-                <mesh filename="package://pentaslam_description/meshes/ROBOT_ASSEMBLY.stl" scale="0.001 0.001 0.001"/>
+                <mesh filename="package://slambot_description/meshes_version_2/ROBOT_ASSEMBLY.stl" scale="0.001 0.001 0.001"/>
             </geometry>
         </visual>
@@ -29,5 +31,5 @@
             <origin xyz="0 0 0" rpy="0 0 0"/>
             <geometry>
-                <mesh filename="package://pentaslam_description/meshes/ROBOT_ASSEMBLY.stl" scale="0.001 0.001 0.001"/>
+                <mesh filename="package://slambot_description/meshes_version_2/ROBOT_ASSEMBLY.stl" scale="0.001 0.001 0.001"/>
             </geometry>
         </collision>
@@ -37,5 +39,5 @@
         <parent link="chassis"/>
         <child link="castor_link1"/>
-    <origin xyz="-0.06580 0.0657 -0.062" rpy="0.0 0.0 3.142"/>
+        <origin xyz="-0.06580 0.0657 -0.062" rpy="0.0 0.0 3.142"/>
     </joint>
     <link name="castor_link1">
@@ -44,5 +46,5 @@
             <origin xyz="0 0 0" rpy="0 0 0"/>
             <geometry>
-                <mesh filename="package://pentaslam_description/meshes/Eye_Ball.stl" scale="0.001 0.001 0.001"/>
+                <mesh filename="package://slambot_description/meshes_version_2/Eye_Ball.stl" scale="0.001 0.001 0.001"/>
             </geometry>
         </visual>
@@ -50,5 +52,5 @@
             <origin xyz="0 0 0" rpy="0 0 0"/>
             <geometry>
-                <mesh filename="package://pentaslam_description/meshes/Eye_Ball.stl" scale="0.001 0.001 0.001"/>
+                <mesh filename="package://slambot_description/meshes/Eye_Ball.stl" scale="0.001 0.001 0.001"/>
             </geometry>
         </collision>
@@ -65,5 +67,5 @@
             <origin xyz="0 0 0" rpy="0 0 0"/>
             <geometry>
-                <mesh filename="package://pentaslam_description/meshes/Eye_Ball.stl" scale="0.001 0.001 0.001"/>
+                <mesh filename="package://slambot_description/meshes/Eye_Ball.stl" scale="0.001 0.001 0.001"/>
             </geometry>
         </visual>
@@ -71,5 +73,5 @@
             <origin xyz="0 0 0" rpy="0 0 0"/>
             <geometry>
-                <mesh filename="package://pentaslam_description/meshes/Eye_Ball.stl" scale="0.001 0.001 0.001"/>
+                <mesh filename="package://slambot_description/meshes/Eye_Ball.stl" scale="0.001 0.001 0.001"/>
             </geometry>
         </collision>
@@ -87,5 +89,5 @@
             <origin xyz="0 0 0" rpy="0 0 0"/>
             <geometry>
-                <mesh filename="package://pentaslam_description/meshes/85mm_Wheel.stl" scale="0.001 0.001 0.001"/>
+                <mesh filename="package://slambot_description/meshes/85mm_Wheel.stl" scale="0.001 0.001 0.001"/>
             </geometry>
         </visual>
@@ -93,5 +95,5 @@
             <origin xyz="0 0 0" rpy="0 0 0"/>
             <geometry>
-                <mesh filename="package://pentaslam_description/meshes/85mm_Wheel.stl" scale="0.001 0.001 0.001"/>
+                <mesh filename="package://slambot_description/meshes/85mm_Wheel.stl" scale="0.001 0.001 0.001"/>
             </geometry>
         </collision>
@@ -109,5 +111,5 @@
             <origin xyz="0 0 0" rpy="0 0 0"/>
             <geometry>
-                <mesh filename="package://pentaslam_description/meshes/85mm_Wheel.stl" scale="0.001 0.001 0.001"/>
+                <mesh filename="package://slambot_description/meshes/85mm_Wheel.stl" scale="0.001 0.001 0.001"/>
             </geometry>
         </visual>
@@ -115,5 +117,5 @@
             <origin xyz="0 0 0" rpy="0 0 0"/>
             <geometry>
-                <mesh filename="package://pentaslam_description/meshes/85mm_Wheel.stl" scale="0.001 0.001 0.001"/>
+                <mesh filename="package://slambot_description/meshes/85mm_Wheel.stl" scale="0.001 0.001 0.001"/>
             </geometry>
         </collision>
@@ -130,5 +132,5 @@
             <origin xyz="0 0 0" rpy="0 0 0"/>
             <geometry>
-                <mesh filename="package://pentaslam_description/meshes/LidarTop.stl" scale="0.001 0.001 0.001"/>
+                <mesh filename="package://slambot_description/meshes/LidarTop.stl" scale="0.001 0.001 0.001"/>
             </geometry>
         </visual>
@@ -136,5 +138,5 @@
             <origin xyz="0 0 0" rpy="0 0 0"/>
             <geometry>
-                <mesh filename="package://pentaslam_description/meshes/LidarTop.stl" scale="0.001 0.001 0.001"/>
+                <mesh filename="package://slambot_description/meshes/LidarTop.stl" scale="0.001 0.001 0.001"/>
             </geometry>
         </collision>
@@ -151,5 +153,5 @@
             <origin xyz="0 0 0" rpy="0 0 0"/>
             <geometry>
-                <mesh filename="package://pentaslam_description/meshes/MPU60501.stl" scale="0.001 0.001 0.001"/>
+                <mesh filename="package://slambot_description/meshes/MPU60501.stl" scale="0.001 0.001 0.001"/>
             </geometry>
         </visual>
@@ -157,5 +159,5 @@
             <origin xyz="0 0 0" rpy="0 0 0"/>
             <geometry>
-                <mesh filename="package://pentaslam_description/meshes/MPU60501.stl" scale="0.001 0.001 0.001"/>
+                <mesh filename="package://slambot_description/meshes/MPU60501.stl" scale="0.001 0.001 0.001"/>
             </geometry>
         </collision>

File: src/slambot_description/urdf/pentaslam_gazebo.xacro (robot description, xacro)
@@ -1,7 +1,7 @@
 <?xml version="1.0"?>
-<robot name="pentaslam"
+<robot name="slambot"
     xmlns:xacro="http://ros.org/wiki/xacro">
     <gazebo>
-        <plugin name="libgazebo_ros2_control.so" filename="gazebo_ros2_control">
+        <plugin filename="libgazebo_ros2_control.so" name="gazebo_ros2_control">
             <robot_param>robot_description</robot_param>
             <robot_param_node>robot_state_publisher</robot_param_node>

Commit message: Commit

File: src/slambot_description/urdf/pentaslam.urdf.xacro (robot description, xacro)
@@ -14,11 +14,12 @@
         </inertial>
     </xacro:macro>
-    <link name="base_link"/>
-    <joint name="joint_name" type="fixed">
-        <parent link="base_link"/>
-        <child link="chassis"/>
-        <origin xyz="0.0 0.0 0.07" rpy="0.0 0.0 3.142"/>
+    <link name="base_footprint"/>
+    <joint name="base_joint" type="fixed">
+        <parent link="base_footprint"/>
+        <child link="base_link"/>
+        <axis xyz="0 0 0"/>
+        <origin xyz="0 0 0" rpy="0 0 0"/>
     </joint>
-    <link name="chassis">
+    <link name="base_link">
         <xacro:default_inertial mass="1.0"/>
         <visual>
@@ -37,5 +38,5 @@
     <!-- CASTOR WHEEL1 LINK -->
     <joint name="caster_wheel_joint1" type="fixed">
-        <parent link="chassis"/>
+        <parent link="base_link"/>
         <child link="castor_link1"/>
         <origin xyz="-0.06580 0.0657 -0.062" rpy="0.0 0.0 3.142"/>
@@ -58,5 +59,5 @@
     <!-- CASTOR WHEEL2 LINK -->
     <joint name="caster_wheel_joint2" type="fixed">
-        <parent link="chassis"/>
+        <parent link="base_link"/>
         <child link="castor_link2"/>
         <origin xyz="-0.06640 -0.0425 -0.062" rpy="0.0 0.0 3.142"/>
@@ -79,5 +80,5 @@
     <!-- LEFT WHEEL LINK -->
     <joint name="left_wheel_joint" type="continuous">
-        <parent link="chassis"/>
+        <parent link="base_link"/>
         <child link="left_wheel"/>
         <origin xyz="0.074757 -0.120900 -0.024" rpy="0.0 0.0 3.142"/>
@@ -101,5 +102,5 @@
     <!-- RIGHT WHEEL LINK -->
     <joint name="right_wheel_joint" type="continuous">
-        <parent link="chassis"/>
+        <parent link="base_link"/>
         <child link="right_wheel"/>
         <origin xyz="0.074757 0.126900 -0.024" rpy="0.0 0.0 0.0"/>
@@ -123,5 +124,5 @@
     <!-- LIDAR LINK-->
     <joint name="lidar_joint" type="fixed">
-        <parent link="chassis"/>
+        <parent link="base_link"/>
         <child link="lidar"/>
         <origin xyz="0.08100009757 0.005 0.0988" rpy="0.0 0.0 1.57"/>
@@ -144,5 +145,5 @@
     <!-- IMU_LINK -->
     <joint name="imu_joint" type="fixed">
-        <parent link="chassis"/>
+        <parent link="base_link"/>
         <child link="imu"/>
         <origin xyz="0.0002 0.0084 0.0766" rpy="1.57 0.0 -1.57"/>
